File: rak-module-board/rak-module-board.kicad_sch (KiCad schematic)
At the start: 66 parts, among them J1 20449-001E-03, J2 20449-001E-03, U1 SX1262IMLTRT, U2 PE42359SCAA-Z, U3 32MHz, U4 NRF52840-QIAA, Y2 32.768K

Commit message: Add files via upload
Parts:
- removed C24: NC, symbol Device:C
- removed C29: 12pF, symbol Device:C
- removed R7: NC, symbol Device:R
- added BT1: Battery_Cell, symbol Device:Battery_Cell
- added BT2: Battery_Cell, Battery:BatteryHolder_Keystone_2460_1xAA, symbol Device:Battery_Cell
- added C26, C45: NC, symbol Device:C
- added C44, C47, C48, C49, C50, C51, C52, C53, C54, C55, C56, C57, C61, C62, C63, C64, C65, C66, C67, C68, C69, C80, C81, C82, C83, C85, C87, C89, C90, C91: 100nF, symbol Device:C
- added C46, C84: 10uF, symbol Device:C
- added C58, C70, C88: 1uF, symbol Device:C
- added C59, C60: 100uF, symbol Device:C
- added C71, C74: 22pF, symbol Device:C
- added C72, C73: 12pF, symbol Device:C
- added C76, C77: 300pF, symbol Device:C
- added C78: 11mF, symbol Device:C_Polarized
- added C79: 70mF, symbol Device:C_Polarized
- added C86: 100pF, symbol Device:C
- added D2, D3, D4: MBR140SFT1G, symbol Device:D_Schottky
- added D5: RED, symbol Device:LED
- added D6: GREEN, symbol Device:LED
- added D7: BLUE, symbol Device:LED
- added H1, H2, H3, H4: MountingHole, symbol Mechanical:MountingHole
- added J3: 2171840001, 2171840001_MOL, symbol 2023-02-17_09-35-09:2171840001
- added J4: 20449-001E-03, MHF 4_RECE_IPX, symbol 2023-02-13_21-49-33:20449-001E-03
- added L11: 4.7uH, symbol Device:L_Iron
- added L12: 2.2uH, symbol Device:L_Iron
- added L14: NC, symbol Device:L
- added L15: 47nH, symbol Device:L
- added L16: 120uH, symbol Device:L_Iron
- added LS1: MLT-8530, MLT-8530_JHE, symbol 2023-02-20_17-21-59:MLT-8530
- added Q1, Q2: NCE40P40K, TO-252_WUX, symbol 2023-02-16_20-52-39:NCE40P40K
- added Q3, Q4: DTC143Z, symbol Transistor_BJT:DTC143Z
- added R10, R13, R15, R43, R45, R54, R56, R57, R64, R65, R66, R67, R8: NC, symbol Device:R
- added R11, R12, R14, R41, R42, R51, R55, R58, R59, R63, R9: 0, symbol Device:R
- added R16: 47K, symbol Device:R
- added R17, R19, R32: 100K, symbol Device:R
- added R18, R33, R34, R48, R49, R50, R52: 10K, symbol Device:R
- added R20, R29: 1M, symbol Device:R
- added R21, R28: 1.5M, symbol Device:R
- added R22: 1k, symbol Device:R
- added R23: 2.7k, symbol Device:R
- added R24, R25: 4.7k, symbol Device:R
- added R26: 100k, symbol Device:R
- added R27: 800k, symbol Device:R
- added R30: 32.4K, symbol Device:R
- added R31: 2K, symbol Device:R
- added R35, R36, R37, R38, R47, R61, R62: 4.7K, symbol Device:R
- added R39, R40: 1K, symbol Device:R
- added R46: 330, symbol Device:R
- added R53: 100, symbol Device:R
- added R60: 10, symbol Device:R
- added SW1: SS-12D10G5, SS-12D10G5_XKB, symbol 2023-02-17_08-25-45:SS-12D10G5
- added SW2: SW_DPST_x2, symbol Switch:SW_DPST_x2
- added TP1, TP10, TP11, TP12, TP2, TP3, TP4, TP5, TP6, TP7, TP8, TP9: TestPoint, symbol Connector:TestPoint
- added U10: LRC399-04AT1G, symbol power.vbat_sx_sym:LRC399-04AT1G
- added U11: SCD30, symbol power.vbat_sx_sym:SCD30
- added U12, U6: MMBT4401LT1G, SOT-23_ONS, symbol 2023-02-16_21-03-21:MMBT4401LT1G
- added U13: RV-3028-C7_32.768KHZ_1PPM-TA-QA, RV-3028-C7_MCX, symbol 2023-02-20_17-57-05:RV-3028-C7_32.768KHZ_1PPM-TA-QA
- added U14: SHTC3, SHTC3_SEN, symbol 2023-02-20_22-04-55:SHTC3
- added U15: BME680, Package_LGA:Bosch_LGA-8_3x3mm_P0.8mm_ClockwisePinNumbering, symbol Sensor:BME680
- added U16: MAX-8Q-0, ARRAY_X-8Q-0_UBL, symbol 2023-02-21_16-36-23:MAX-8Q-0
- added U5: AT25QL321-MBUE-T, AT25QL321-MBUE-T_ADO, symbol 2023-02-15_08-42-47:AT25QL321-MBUE-T
- added U7: TP4054ST25K, SOT-23-5L_TPW, symbol 2023-02-17_08-42-11:TP4054ST25K
- added U8: SGM6036-ADJ, symbol power.vbat_sx_sym:SGM6036-ADJ
- added U9: SGM6019, symbol power.vbat_sx_sym:SGM6019
- added Y1: 32MHz, symbol Device:Crystal
- L13: renamed from L; value 120 -> 120uH
- renumbered C8 to C75
Connections:
- net +BATT: now also BT1.1 (+), BT2.1 (+), C49.1, C50.1, C51.1, C52.1, C55.1, C56.1, C57.1, C57.2, C58.1, C59.1, C60.1, C61.1, C62.1, C65.1, C66.1, D2.1 (K), D3.1 (K), D4.1 (K), D5.2 (A), Q1.2, Q1.3, Q2.1, Q2.2, Q2.3, R11.2, R12.2, R13.2, R14.1, R14.2, R15.1, R15.2, R16.1, R17.2, R19.1, R20.1, R26.1, R33.1, R39.1, R40.1, R8.2, SW1.1, SW1.2, SW1.3, U7.3 (BAT), U7.4 (VCC), U8.6 (VIN), U9.1 (VIN)
- net GND: now also C32.2, C33.2, J1.2, J2.2, U4.74 (VSS), BT1.2 (-), BT2.2 (-), C26.2, C44.2, C45.2, C46.2, C47.2, C48.2, C49.2, C50.2, C51.2, C52.2, C53.2, C54.2, C55.2, C56.2, C58.2, C59.2, C60.2, C61.2, C62.2, C63.2, C64.2, C65.2, C66.2, C67.2, C68.2, C69.2, C70.2, C72.2, C73.2, C76.2, C77.2, C78.2, C79.2, C80.2, C81.2, C82.2, C83.2, C84.2, C85.2, C87.2, C88.2, C89.2, C90.2, C91.2, D4.2 (A), J3.A1 (GND), J3.A12 (GND), J3.B1 (GND), J3.B12 (GND), J4.1, J4.2, J4.3, Q3.2 (E), Q4.2 (E), R18.2, R19.2, R21.2, R23.2, R24.1, R25.2, R29.2, R30.2, R47.2, R55.2, R67.2, SW2.1 (A), TP6.1, U10.2 (GND), U11.2 (GND), U11.7 (SEL), U12.2 (EMITTER), U13.5 (VSS), U14.4 (VSS), U15.1 (GND), U15.7 (GND), U16.1 (GND), U16.10 (GND), U16.12 (GND), U5.4, U6.2 (EMITTER), U7.2 (GND), U8.4 (GND), U8.7 (EXPAD), U9.5 (SGND), U9.7 (PGND), U9.9 (EXPAD); no longer J1.4, J2.4
- net LED1: now also Q3.1 (B)
- net LED2: now also Q4.1 (B)
- net NFC1: now also C76.1, L14.2, R42.1
- net NFC2: now also C77.1, L14.1, R41.1
- net NRF_RESET: now also C44.1, R34.2
- net PO-04/AIN2: now also R48.2, TP4.1, U13.2 (INT), U16.4 (TIMEPULSE)
- net QSPI_CLK: now also U5.6
- net QSPI_CS: now also U5.1
- net QSPI_DIO1: now also U5.2
- net QSPI_DIO2: now also U5.3
- net QSPI_DIO3: now also U5.7
- net RF_BT: now also R43.2
- net UART1_DE: now also R63.1, R64.1, TP5.1, U13.1 (CLKOUT)
- net UART1_RX: now also TP8.1, U16.2 (TXD)
- net UART1_TX: now also TP9.1, U16.3 (RXD)
- net VBUS: now also D2.2 (A), J3.A4 (VBUS), J3.A9 (VBUS), J3.B4 (VBUS), J3.B9 (VBUS)
- net VDD: now also C80.1, R10.2, R48.1, R49.1, R50.1, R51.2, R52.1, R53.1, R8.1, U13.7 (VDD)
- net at C35.1, C36.1, L9.2: now also J2.4, R43.1; no longer J2.2
- net at C12.1, L4.2, R2.1: now also J1.4; no longer J1.2
- net at U4.A18 (DEC2): now also C26.1
- net at U4.B24 (XC1): now also C73.1, Y1.1
- net at U4.A23 (XC2): now also C72.1, Y1.2
- net PO-30/AIN6 renamed QSPI_DIO0
- net QSPI_DIO0: now also U5.5
- net QC_SCL renamed I2C_SCL
- net I2C_SCL: now also R35.2, R49.2, R57.1, R66.1, TP12.1, TP3.1, U11.3 (TX/SCL), U13.3 (SCL), U14.2 (SCL), U15.4 (SCK)
- net QC_SCL_2 renamed I2C_SCL_2
- net I2C_SCL_2: now also R37.2
- net QC_SDA renamed I2C_SDA
- net I2C_SDA: now also R36.2, R50.2, R56.1, R65.1, TP11.1, TP2.1, U11.4 (RX/SDA), U13.4 (SDA), U14.3 (SDA), U15.3 (SDI)
- net QC_SDA_2 renamed I2C_SDA_2
- net I2C_SDA_2: now also R38.2
- new net: R52.2, TP1.1, U13.8 (EVI)
- new net: D5.1 (K), R22.1
- new net: J3.B5 (CC2), R25.1
- new net: R54.2, R55.1, U15.5 (SDO)
- new net: J3.A5 (CC1), R24.2
- new net: R45.2, R46.2, R47.1, U12.1 (BASE)
- new net: LS1.2, U12.3 (COLLECTOR)
- new net: C71.1, R27.1, R29.1, U8.3 (OUT)
- new net: R27.2, R28.1
- new net: C86.1, U16.11 (RF_IN)
- new net: C86.2, J4.4, L15.2
- new net: Q1.1, R17.1, U6.3 (COLLECTOR)
- new net: R60.1, U16.14 (VCC_RF)
- new net: L15.1, R60.2
- new net: R33.2, R67.1, U9.4 (MODE)
- new net: C74.1, R30.1, R31.1, U9.6 (FB)
- new net: L12.1, U9.8 (SW)
- new net: C70.1, R26.2, U8.5 (EN)
- new net: D6.2 (A), R39.2
- new net: D7.1 (K), Q4.3 (C)
- new net: D7.2 (A), R40.2
- new net: C78.1, C79.1, R53.2, U13.6 (VBACKUP)
- new net: D6.1 (K), Q3.3 (C)
- new net: R58.2, U16.6 (V_BCKP)
- new net: R59.2, U16.7 (VCC_IO)
- new net: R16.2, R18.1, U6.1 (BASE)
- new net: C85.1, R59.1
- new net: L11.1, U8.2 (SW)
- new net: R23.1, U7.5 (PROG)
- new net: R31.2, R32.1
- new net: R22.2, U7.1 (*CHRG)
- new net: C84.1, R58.1
- new net +3V3: C45.1, C46.1, C47.1, C48.1, C63.1, C64.1, C67.1, C68.1, C71.2, C74.2, C81.1, C82.1, C83.1, C87.1, C89.1, C90.1, C91.1, L11.2, L12.2, L16.1, L16.2, LS1.1, R10.1, R11.1, R12.1, R13.1, R28.2, R32.2, R34.1, R35.1, R36.1, R37.1, R38.1, R51.1, R54.1, R56.2, R57.2, R61.1, R62.1, R65.2, R66.2, R9.1, TP10.1, TP7.1, U11.1 (VDD), U14.1 (VDD), U15.2 (CSB), U15.6 (VDDIO), U15.8 (VDD), U16.8 (VCC)
- new net ADC_VBAT: R20.2, R21.1
- new net IO2: U9.2 (EN)
- new net IO5: R42.2, R46.1, U11.6 (PWM)
- new net IO6: R41.2, R45.1, U11.5 (RDY)
- new net RESET: C69.1, SW2.2 (B)
- new net RESET_GPS: C88.1, R62.2, R63.2, U16.9 (RESET_IN)
- new net STANDBY: R61.2, R64.2, U16.5 (EXTINT)
- new net USB N: J3.A7 (DN1), J3.B7 (DN2), U10.4 (I/O4)
- new net USB P: J3.A6 (DP1), J3.B6 (DP2), U10.6 (I/O3)
- new net VCC: D3.2 (A)
- new net VD: C53.1, C54.1, R9.2, U5.8
- no-connect marks 12 -> 33
Other:
- moved on the sheet: C11, C12, C13, C14, C19, C20, C21, C22, C23, C25, C27, C28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

Commit message: Add files via upload
Parts:
- removed BT1: Battery_Cell, symbol Device:Battery_Cell
- removed BT2: Battery_Cell, Battery:BatteryHolder_Keystone_2460_1xAA, symbol Device:Battery_Cell
- removed C51, C52: 100nF, symbol Device:C
- removed C78: 11mF, symbol Device:C_Polarized
- removed C79: 70mF, symbol Device:C_Polarized
- removed R53: 100, symbol Device:R
- removed SW1: SS-12D10G5, SS-12D10G5_XKB, symbol 2023-02-17_08-25-45:SS-12D10G5
- added B1: BHC-18650-1P, footprints:BHC-18650-1P, symbol 2023-02-23_11-19-04:BHC-18650-1P
- C10, C11, C12, C13, C14, C15, C16, C17, C18, C19, C2, C20, C21, C22, C23, C25, C26, C27, C28, C3, C30, C31, C32, C33, C34, C35, C36, C37, C38, C39, C4, C40, C41, C42, C43, C44, C45, C46, C47, C48, C49, C5, C50, C53, C54, C55, C56, C57, C58, C59, C6, C60, C61, C62, C63, C64, C65, C66, C67, C68, C69, C7, C70, C71, C72, C73, C74, C75, C76, C77, C8, C80, C81, C82, C83, C84, C85, C86, C87, C88, C89, C9, C90, C91: footprint (none) -> Capacitor_SMD:C_0603_1608Metric_Pad1.08x0.95mm_HandSolder
- D2, D3, D4: footprint (none) -> footprints:MBR140SFT1G
- D5, D6, D7: footprint (none) -> LED_SMD:LED_0603_1608Metric_Pad1.05x0.95mm_HandSolder
- H1, H2, H3, H4: footprint (none) -> MountingHole:MountingHole_2.7mm
- J1, J2, J4: footprint MHF 4_RECE_IPX -> footprints:20449-001E-03
- J3: footprint 2171840001_MOL -> footprints:2171840001
- L1, L11, L12, L13, L14, L15, L2, L3, L4, L6, L7, L9: footprint (none) -> Inductor_SMD:L_0201_0603Metric_Pad0.64x0.40mm_HandSolder
- L10, L5, L8: footprint (none) -> Inductor_SMD:L_0805_2012Metric_Pad1.05x1.20mm_HandSolder
- L16: footprint (none) -> Inductor_SMD:L_1008_2520Metric_Pad1.43x2.20mm_HandSolder
- LS1: footprint MLT-8530_JHE -> footprints:MLT-8530
- Q1, Q2: footprint TO-252_WUX -> footprints:NCE40P40K
- Q3, Q4: footprint (none) -> footprints:DTC143ZEBTL
- R1, R10, R11, R12, R13, R14, R15, R16, R17, R18, R19, R2, R20, R21, R22, R23, R24, R25, R26, R27, R28, R29, R3, R30, R31, R32, R33, R34, R35, R36, R37, R38, R39, R40, R41, R42, R43, R45, R46, R47, R48, R49, R5, R50, R51, R52, R54, R55, R56, R57, R58, R59, R6, R60, R61, R62, R63, R64, R65, R66, R67, R8, R9: footprint (none) -> Resistor_SMD:R_0201_0603Metric_Pad0.64x0.40mm_HandSolder
- SW2: footprint (none) -> Button_Switch_SMD:SW_Push_1P1T_NO_CK_KMR2
- TP1, TP10, TP11, TP12, TP2, TP3, TP4, TP5, TP6, TP7, TP8, TP9: footprint (none) -> TestPoint:TestPoint_Pad_D1.0mm
- U1: footprint QFN24_4X4_SEM -> footprints:SX1262IMLTRT
- U10: footprint (none) -> Package_SO:TSOP-6_1.65x3.05mm_P0.95mm
- U11: footprint (none) -> footprints:MODULE_SCD30
- U12, U6: footprint SOT-23_ONS -> footprints:MMBT4401LT1G
- U13: footprint RV-3028-C7_MCX -> footprints:RV-3028-C7 32.768KHZ 1PPM-TA-QA
- U14: footprint SHTC3_SEN -> footprints:SHTC3
- U15: footprint Package_LGA:Bosch_LGA-8_3x3mm_P0.8mm_ClockwisePinNumbering -> footprints:BME680
- U16: footprint ARRAY_X-8Q-0_UBL -> footprints:MAX-8Q-0
- U2: footprint SC-70-6_PSM -> footprints:PE42359SCAA-Z
- U4: footprint AQFN73_7X7_NOR -> footprints:NRF52840-QIAA-R
- U5: footprint AT25QL321-MBUE-T_ADO -> footprints:AT25QL321-MBUE-T
- U7: footprint SOT-23-5L_TPW -> footprints:TP4054ST25K
- U8: footprint (none) -> footprints:SGM6036-ADJ
- U9: footprint (none) -> Package_DFN_QFN:TDFN-8-1EP_3x2mm_P0.5mm_EP1.4x1.4mm
- Y1: footprint (none) -> Crystal:Crystal_SMD_5032-2Pin_5.0x3.2mm
- Y2: footprint (none) -> Crystal:Crystal_SMD_MicroCrystal_CC4V-T1A-2Pin_5.0x1.9mm_HandSoldering
Connections:
- net +BATT: now also B1.2
- net GND: now also B1.1
- no-connect marks 33 -> 34
Other:
- moved on the sheet: C49, C50, C53, C54, C80

Commit message: Add files via upload
Connections:
- net IO2 is gone; now on net SW2: U9.2 (EN)
- net RESET is gone; now on net NRF_RESET: C69.1, SW2.2 (B)
Changed lines of the file:
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@@
     (effects (font (size 1.27 1.27)) (justify right bottom))
   )
-  (label "IO2" (at 133.604 145.288 0)
+  (label "SW2" (at 133.604 145.288 0)
     (effects (font (size 1.27 1.27)) (justify left bottom))
   )
@@
     (effects (font (size 1.27 1.27)) (justify right bottom))
   )
-  (label "RESET" (at 350.774 22.86 180)
+  (label "NRF_RESET" (at 350.774 22.86 180)
     (effects (font (size 1.27 1.27)) (justify right bottom))
   )

Commit message: Add files via upload
Connections:
- net NRF_USB+ is gone; now on net USB P: U4.AD6 (D+)
- net NRF_USB- is gone; now on net USB N: U4.AD4 (D-)
- net PO-05/AIN3 is gone; now on net ADC_VBAT: U4.K2 (P0-05/AIN3)
Changed lines of the file:
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@@
     (effects (font (size 1.27 1.27)) (justify right bottom))
   )
-  (label "NRF_USB+" (at 91.694 265.684 0)
+  (label "USB P" (at 91.694 265.684 0)
     (effects (font (size 1.27 1.27)) (justify left bottom))
   )
@@
     (effects (font (size 1.27 1.27)) (justify left bottom))
   )
-  (label "PO-05{slash}AIN3" (at 91.694 207.264 0)
+  (label "ADC_VBAT" (at 91.694 207.264 0)
     (effects (font (size 1.27 1.27)) (justify left bottom))
   )
@@
     (effects (font (size 1.27 1.27)) (justify right bottom))
   )
-  (label "NRF_USB-" (at 91.694 263.144 0)
+  (label "USB N" (at 91.694 263.144 0)
     (effects (font (size 1.27 1.27)) (justify left bottom))
   )
