File: rak-module-board/rak-module-board.kicad_pcb (KiCad board)
At the start: 2 copper layers, 99.1 x 99.1 mm, 214 parts, among them J1 20449-001E-03, J2 20449-001E-03, J3 2171840001, J4 20449-001E-03, Q1 NCE40P40K, Q2 NCE40P40K, Q3 DTC143Z, Q4 DTC143Z, SW2 SW_DPST_x2, U1 SX1262IMLTRT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

Commit message: Add files via upload
Parts:
- moved J1 289.8 mm to (152.4, 44.5), turned to 180 degrees
- moved R65 289.6 mm to (195.6, 77.5), turned to 180 degrees
- moved R66 289.1 mm to (193.0, 74.9), turned to 90 degrees
- moved R52 285.6 mm to (191.8, 86.4), turned to 90 degrees
- moved R50 273.1 mm to (191.8, 94.0), turned to -90 degrees
- moved C15 266.6 mm to (156.2, 61.6), turned to -90 degrees
- moved R67 263.8 mm to (166.4, 72.4)
- moved C57 252.2 mm to (156.2, 126.1), turned to -90 degrees
- moved C8 248.7 mm to (156.2, 66.3), turned to 90 degrees
- moved C45 245.0 mm to (149.9, 108.0)
- moved C48 243.5 mm to (145.5, 108.0), turned to 180 degrees
- moved D3 233.7 mm to (133.3, 116.8)
- moved R18 228.6 mm to (152.4, 128.9)
- moved R9 228.1 mm to (129.8, 81.3), turned to 90 degrees
- moved R11 227.1 mm to (127.0, 78.7), turned to 90 degrees
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Connections:
- C69 pad 1: /RESET -> /NRF_RESET
- SW2 pad 2: /RESET -> /NRF_RESET
- U9 pad 2: /IO2 -> /SW2

Commit message: Add files via upload
Parts:
- moved TP5 2.79 mm to (199.4, 85.3)
- moved TP4 2.54 mm to (199.4, 87.6)
- moved TP3 2.29 mm to (199.4, 89.9)
- moved TP1 2.03 mm to (199.4, 92.2)
- moved TP2 1.78 mm to (199.4, 94.5)
- moved R58 0.96 mm to (195.1, 55.2), turned to -90 degrees
- moved R14 0.61 mm to (129.8, 75.6)
- moved R15 0.61 mm to (128.3, 75.6)
- moved R11 0.33 mm to (127.0, 78.4)
- moved R12 0.33 mm to (128.3, 78.4)
- moved R13 0.33 mm to (129.8, 78.4)
- moved C74 0.25 mm to (171.7, 69.8)
- moved R66 0.25 mm to (192.8, 74.9)
- turned J1 to 0 degrees
- turned J4 to -90 degrees
Connections:
- U4 pad AD4: /NRF_USB- -> /USB N
- U4 pad AD6: /NRF_USB+ -> /USB P
- U4 pad K2: /PO-05/AIN3 -> /ADC_VBAT
Routing:
- net GND: track 0.00 -> 709.2 mm, vias 0 -> 55
- net +3V3: track 0.00 -> 345.1 mm, vias 0 -> 30
- net +BATT: track 0.00 -> 294.1 mm, vias 0 -> 17
- net /I2C_SDA: track 0.00 -> 176.6 mm, vias 0 -> 13
- net /PO-04/AIN2: track 0.00 -> 153.1 mm, vias 0 -> 11
- net VDD: track 0.00 -> 151.7 mm, vias 0 -> 15
- net /I2C_SCL: track 0.00 -> 142.1 mm, vias 0 -> 11
- net VBUS: track 0.00 -> 125.8 mm, vias 0 -> 12
- net /UART1_TX: track 0.00 -> 108.4 mm, vias 0 -> 8
- net /USB N: track 0.00 -> 90.4 mm, vias 0 -> 6
- net /USB P: track 0.00 -> 87.1 mm, vias 0 -> 7
- net Net-(C35-Pad1): track 0.00 -> 80.2 mm, vias 0 -> 10
- net Net-(C3-Pad2): track 0.00 -> 56.0 mm, vias 0 -> 4
- net /NFC1: track 0.00 -> 52.1 mm, vias 0 -> 4
- net /SW2: track 0.00 -> 43.4 mm, vias 0 -> 4
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
Commit message: Add files via upload
Parts:
- U13: value RV-3028-C7_32.768KHZ_1PPM-TA-QA -> RV-3028-C7
Routing:
- net /UART1_DE: track 11.4 -> 128.7 mm, vias 3 -> 7
- net /UART1_RX: track 15.5 -> 122.8 mm, vias 2 -> 8
- net /NRF_RESET: track 20.4 -> 103.6 mm, vias 4 -> 8
- net /ADC_VBAT: track 1.72 -> 78.3 mm, vias 0 -> 6
- net /DEC4_6: track 29.1 -> 79.4 mm, vias 2 -> 6
- net /DIO2: track 0.00 -> 44.5 mm, vias 0 -> 5
- net Net-(C35-Pad1): track 80.2 -> 117.9 mm, vias 10 -> 9
- net Net-(C13-Pad1): track 6.24 -> 42.4 mm, vias 0 -> 4
- net /LED1: track 0.00 -> 30.6 mm, vias 0 -> 4
- net /I2C_SCL: track 142.1 -> 172.0 mm
- net Net-(C34-Pad1): track 0.00 -> 29.8 mm, vias 0 -> 2
- net Net-(C33-Pad1): track 0.00 -> 23.6 mm, vias 0 -> 2
- net VDD: track 151.7 -> 173.2 mm, vias 15 -> 18
- net VBUS: track 125.8 -> 107.0 mm
- net /QSPI_DIO2: track 0.00 -> 18.2 mm, vias 0 -> 4
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
Commit message: Add files via upload
Routing:
- net +3V3: vias 30 -> 29
Changed lines of the file:
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@@
   (segment (start 131.4715 135.0275) (end 131.572 135.128) (width 0.254) (layer "F.Cu") (net 16))
   (segment (start 129.54 135.0275) (end 131.4715 135.0275) (width 0.254) (layer "F.Cu") (net 16))
+  (segment (start 124.689 78.003) (end 124.46 78.232) (width 0.254) (layer "F.Cu") (net 16))
   (segment (start 146.304 120.7135) (end 146.304 115.9637) (width 0.254) (layer "F.Cu") (net 16))
   (segment (start 147.066 65.024) (end 148.59 63.5) (width 0.254) (layer "F.Cu") (net 16))
@@
   (segment (start 127 132.4875) (end 127.4075 132.08) (width 0.254) (layer "F.Cu") (net 16))
   (segment (start 142.8115 73.140001) (end 141.974001 73.140001) (width 0.254) (layer "F.Cu") (net 16))
-  (segment (start 124.689 78.003) (end 124.46 78.232) (width 0.254) (layer "F.Cu") (net 16))
+  (segment (start 127 78.003) (end 124.689 78.003) (width 0.254) (layer "F.Cu") (net 16))
   (segment (start 162.7135 99.9225) (end 162.56 100.076) (width 0.254) (layer "F.Cu") (net 16))
   (segment (start 127.254 109.22) (end 127.254 109.1365) (width 0.254) (layer "F.Cu") (net 16))
@@
   (segment (start 163.4225 74.115) (end 163.4225 72.39) (width 0.254) (layer "F.Cu") (net 16))
   (segment (start 129.8335 78.003) (end 129.8335 75.999) (width 0.254) (layer "F.Cu") (net 16))
-  (segment (start 127 78.003) (end 124.689 78.003) (width 0.254) (layer "F.Cu") (net 16))
   (segment (start 134.6985 66.294) (end 135.36 65.6325) (width 0.254) (layer "F.Cu") (net 16))
   (segment (start 126.746 111.76) (end 126.1375 111.1515) (width 0.254) (layer "F.Cu") (net 16))
@@
   (via (at 164.084 105.664) (size 0.6) (drill 0.4) (layers "F.Cu" "B.Cu") (net 29))
   (segment (start 165.1 94.488) (end 165.1 93.472) (width 0.2) (layer "B.Cu") (net 29))
-  (segment (start 169.418 105.664) (end 169.418 125.476) (width 0.2) (layer "B.Cu") (net 29))
+  (segment (start 168.656 125.476) (end 169.418 124.714) (width 0.2) (layer "B.Cu") (net 29))
   (segment (start 140.208 133.35) (end 140.208 124.968) (width 0.2) (layer "B.Cu") (net 29))
+  (segment (start 151.384 125.476) (end 168.656 125.476) (width 0.2) (layer "B.Cu") (net 29))
   (segment (start 159.512 105.156) (end 160.02 105.664) (width 0.2) (layer "B.Cu") (net 29))
+  (segment (start 169.418 105.664) (end 169.418 124.714) (width 0.2) (layer "B.Cu") (net 29))
   (segment (start 168.91 89.662) (end 168.91 105.156) (width 0.2) (layer "B.Cu") (net 29))
   (segment (start 159.512 92.71) (end 159.512 105.156) (width 0.2) (layer "B.Cu") (net 29))
   (segment (start 164.084 95.504) (end 165.1 94.488) (width 0.2) (layer "B.Cu") (net 29))
-  (segment (start 169.418 125.476) (end 151.384 125.476) (width 0.2) (layer "B.Cu") (net 29))
   (segment (start 140.208 124.968) (end 140.462 124.714) (width 0.2) (layer "B.Cu") (net 29))
   (segment (start 164.084 105.664) (end 164.084 95.504) (width 0.2) (layer "B.Cu") (net 29))
@@
   (segment (start 148.111851 105.062989) (end 148.528989 105.062989) (width 0.254) (layer "F.Cu") (net 34))
   (segment (start 129.032 78.818) (end 129.8335 78.818) (width 0.254) (layer "F.Cu") (net 34))
-  (segment (start 181.258 131.67) (end 182.118 130.81) (width 0.254) (layer "F.Cu") (net 34))
   (segment (start 175.26 132.08) (end 175.67 131.67) (width 0.254) (layer "F.Cu") (net 34))
   (segment (start 180.34 76.2) (end 182.080901 76.2) (width 0.254) (layer "F.Cu") (net 34))
@@
   (segment (start 185.3195 71.7285) (end 186.442695 71.7285) (width 0.254) (layer "F.Cu") (net 34))
   (segment (start 166.778911 108.557089) (end 166.624 108.712) (width 0.254) (layer "F.Cu") (net 34))
-  (segment (start 177.86 131.67) (end 181.258 131.67) (width 0.254) (layer "F.Cu") (net 34))
   (segment (start 148.876 105.41) (end 148.876 104.720195) (width 0.254) (layer "F.Cu") (net 34))
   (segment (start 171.5505 109.728) (end 171.45 109.6275) (width 0.254) (layer "F.Cu") (net 34))
@@
   (via (at 124.968 112.014) (size 0.6) (drill 0.4) (layers "F.Cu" "B.Cu") (net 34))
   (via (at 168.91 75.692) (size 0.6) (drill 0.4) (layers "F.Cu" "B.Cu") (net 34))
-  (via (at 182.118 130.81) (size 0.6) (drill 0.4) (layers "F.Cu" "B.Cu") (net 34))
   (via (at 147.828 107.95) (size 0.6) (drill 0.4) (layers "F.Cu" "B.Cu") (net 34))
   (via (at 184.404 50.8) (size 0.6) (drill 0.4) (layers "F.Cu" "B.Cu") (net 34))
@@
   (segment (start 139.446 103.82104) (end 139.35148 103.72652) (width 0.254) (layer "B.Cu") (net 34))
   (segment (start 185.42 51.816) (end 184.404 50.8) (width 0.254) (layer "B.Cu") (net 34))
+  (segment (start 181.258 131.67) (end 177.86 131.67) (width 0.254) (layer "B.Cu") (net 34))
   (segment (start 170.942 73.66) (end 170.942 71.882) (width 0.254) (layer "B.Cu") (net 34))
   (segment (start 193.548 74.623) (end 193.6485 74.5225) (width 0.254) (layer "B.Cu") (net 34))
@@
   (segment (start 181.356 86.36) (end 181.61 86.614) (width 0.254) (layer "B.Cu") (net 34))
   (segment (start 185.928 79.375) (end 185.801 79.248) (width 0.254) (layer "B.Cu") (net 34))
+  (segment (start 182.118 130.81) (end 181.258 131.67) (width 0.254) (layer "B.Cu") (net 34))
   (segment (start 125.222 81.788) (end 126.238 80.772) (width 0.254) (layer "B.Cu") (net 34))
   (segment (start 193.548 77.216) (end 193.548 74.623) (width 0.254) (layer "B.Cu") (net 34))
